File: mini-project-2-wled-board.kicad_sch (KiCad schematic)
At the start: 34 parts, among them J101 Conn_01x03, J102 Conn_01x03, J103 Conn_01x03, J104 Conn_01x03, J106 Screw_Terminal_01x02, J3 Conn_02x03_Odd_Even, SW101 SW_SPDT, SW103 SW_Push, SW105 SW_Push, U102 74AHCT1G125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

Commit message: update part numbers
Parts:
- F101: Mouser (none) -> 576-178.6764.0001
- J106: Mouser (none) -> 538-39544-3002
Changed lines of the file:
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@@
   (title_block
     (title "WLED ESP32 Control Board")
-    (date "2023-06-18")
+    (date "2023-10-30")
     (rev "A")
   )
@@
     )
     (property "LCSC" "" (at 139.7 128.27 0)
+      (effects (font (size 1.27 1.27)) hide)
+    )
+    (property "Mouser" "538-39544-3002" (at 139.7 128.27 0)
       (effects (font (size 1.27 1.27)) hide)
     )
@@
       (effects (font (size 1.27 1.27)) hide)
     )
+    (property "Mouser" "576-178.6764.0001" (at 148.59 128.27 0)
+      (effects (font (size 1.27 1.27)) hide)
+    )
