File: usbc-2-0.kicad_sch (KiCad schematic)
At the start: 8 parts, among them J201 USB_C_Receptacle_USB2.0

Commit message: update part numbers
Parts:
- C201: LCSC (none) -> C19702
Changed lines of the file:
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@@
       (effects (font (size 1.27 1.27)) hide)
     )
-    (property "LCSC" "" (at 102.87 43.18 0)
+    (property "LCSC" "C19702" (at 102.87 43.18 0)
       (effects (font (size 1.27 1.27)) hide)
     )
